File: for-split.sch (KiCad schematic (older format))
At the start: 67 parts, among them J1 TRRS, J2 TRRS, U1 ProMicro

Commit message: Add extradata pad and connection
Parts:
- J1, J2: footprint idle-hands:PJ320D_DOUBLESIDED -> Connectors:PJ320D_3.5mm_Jack
- MX0:0, MX0:5: footprint idle-hands:MX_FLIP_CUTOUT -> idle-hands:MX_CUTOUT_VERT_PAD1
- MX0:1, MX0:4: footprint idle-hands:MX_FLIP_CUTOUT -> idle-hands:MX_CUTOUT_VERT_PAD3
- MX0:2, MX0:3, MX1:0, MX1:1, MX1:2, MX1:3, MX1:4, MX1:5, MX2:0, MX2:1, MX2:2, MX2:3, MX2:4, MX2:5, MX3:0, MX3:1, MX3:2, MX3:3, MX3:4, MX3:5, MX4:2, MX4:3: footprint idle-hands:MX_FLIP_CUTOUT -> idle-hands:MX_CUTOUT_VERT
- MX4:0, MX4:5: footprint idle-hands:MX_FLIP_CUTOUT -> idle-hands:MX
- MX4:1, MX4:4: footprint idle-hands:MX_FLIP_CUTOUT -> idle-hands:MX2U_CUTOUT_VERT
- renumbered EXTRADATA to EXTRADATA1
Changed lines of the file:
@@
 F 0 "MX1:0" H 5140 2590 50  0000 C CNN
 F 1 "MX1:11" H 4990 2400 50  0000 C CNN
-F 2 "idle-hands:MX_FLIP_CUTOUT" H 4990 2480 60  0001 C CNN
+F 2 "idle-hands:MX_CUTOUT_VERT" H 4990 2480 60  0001 C CNN
 F 3 "" H 4990 2480 60  0000 C CNN
 	1    4990 2480
@@
 F 0 "MX1:1" H 6040 2590 50  0000 C CNN
 F 1 "MX1:10" H 5890 2400 50  0000 C CNN
-F 2 "idle-hands:MX_FLIP_CUTOUT" H 5890 2480 60  0001 C CNN
+F 2 "idle-hands:MX_CUTOUT_VERT" H 5890 2480 60  0001 C CNN
 F 3 "" H 5890 2480 60  0000 C CNN
 	1    5890 2480
@@
 F 0 "MX1:2" H 6940 2590 50  0000 C CNN
 F 1 "MX1:9" H 6790 2400 50  0000 C CNN
-F 2 "idle-hands:MX_FLIP_CUTOUT" H 6790 2480 60  0001 C CNN
+F 2 "idle-hands:MX_CUTOUT_VERT" H 6790 2480 60  0001 C CNN
 F 3 "" H 6790 2480 60  0000 C CNN
 	1    6790 2480
@@
 F 0 "MX1:3" H 7890 2590 50  0000 C CNN
 F 1 "MX1:8" H 7740 2400 50  0000 C CNN
-F 2 "idle-hands:MX_FLIP_CUTOUT" H 7740 2480 60  0001 C CNN
+F 2 "idle-hands:MX_CUTOUT_VERT" H 7740 2480 60  0001 C CNN
 F 3 "" H 7740 2480 60  0000 C CNN
 	1    7740 2480
@@
 F 0 "MX1:4" H 8840 2590 50  0000 C CNN
 F 1 "MX1:7" H 8690 2400 50  0000 C CNN
-F 2 "idle-hands:MX_FLIP_CUTOUT" H 8690 2480 60  0001 C CNN
+F 2 "idle-hands:MX_CUTOUT_VERT" H 8690 2480 60  0001 C CNN
 F 3 "" H 8690 2480 60  0000 C CNN
 	1    8690 2480
@@
 F 0 "MX0:0" H 5140 1840 50  0000 C CNN
 F 1 "MX0:11" H 4990 1650 50  0000 C CNN
-F 2 "idle-hands:MX_FLIP_CUTOUT" H 4990 1730 60  0001 C CNN
+F 2 "idle-hands:MX_CUTOUT_VERT_PAD1" H 4990 1730 60  0001 C CNN
 F 3 "" H 4990 1730 60  0000 C CNN
 	1    4990 1730
@@
 F 0 "MX0:1" H 6040 1840 50  0000 C CNN
 F 1 "MX0:10" H 5890 1650 50  0000 C CNN
-F 2 "idle-hands:MX_FLIP_CUTOUT" H 5890 1730 60  0001 C CNN
+F 2 "idle-hands:MX_CUTOUT_VERT_PAD3" H 5890 1730 60  0001 C CNN
 F 3 "" H 5890 1730 60  0000 C CNN
 	1    5890 1730
@@
 F 0 "MX0:2" H 6940 1840 50  0000 C CNN
 F 1 "MX0:9" H 6790 1650 50  0000 C CNN
-F 2 "idle-hands:MX_FLIP_CUTOUT" H 6790 1730 60  0001 C CNN
+F 2 "idle-hands:MX_CUTOUT_VERT" H 6790 1730 60  0001 C CNN
 F 3 "" H 6790 1730 60  0000 C CNN
 	1    6790 1730
@@
 F 0 "MX0:3" H 7890 1840 50  0000 C CNN
 F 1 "MX0:8" H 7740 1650 50  0000 C CNN
-F 2 "idle-hands:MX_FLIP_CUTOUT" H 7740 1730 60  0001 C CNN
+F 2 "idle-hands:MX_CUTOUT_VERT" H 7740 1730 60  0001 C CNN
 F 3 "" H 7740 1730 60  0000 C CNN
 	1    7740 1730
@@
 F 0 "MX0:4" H 8840 1840 50  0000 C CNN
 F 1 "MX0:7" H 8690 1650 50  0000 C CNN
-F 2 "idle-hands:MX_FLIP_CUTOUT" H 8690 1730 60  0001 C CNN
+F 2 "idle-hands:MX_CUTOUT_VERT_PAD3" H 8690 1730 60  0001 C CNN
 F 3 "" H 8690 1730 60  0000 C CNN
 	1    8690 1730
@@
 F 0 "MX2:0" H 5140 3340 50  0000 C CNN
 F 1 "MX2:11" H 4990 3150 50  0000 C CNN
-F 2 "idle-hands:MX_FLIP_CUTOUT" H 4990 3230 60  0001 C CNN
+F 2 "idle-hands:MX_CUTOUT_VERT" H 4990 3230 60  0001 C CNN
 F 3 "" H 4990 3230 60  0000 C CNN
 	1    4990 3230
@@
 F 0 "MX2:1" H 6040 3340 50  0000 C CNN
 F 1 "MX2:10" H 5890 3150 50  0000 C CNN
-F 2 "idle-hands:MX_FLIP_CUTOUT" H 5890 3230 60  0001 C CNN
+F 2 "idle-hands:MX_CUTOUT_VERT" H 5890 3230 60  0001 C CNN
 F 3 "" H 5890 3230 60  0000 C CNN
 	1    5890 3230
@@
 F 0 "MX2:2" H 6940 3340 50  0000 C CNN
 F 1 "MX2:9" H 6790 3150 50  0000 C CNN
-F 2 "idle-hands:MX_FLIP_CUTOUT" H 6790 3230 60  0001 C CNN
+F 2 "idle-hands:MX_CUTOUT_VERT" H 6790 3230 60  0001 C CNN
 F 3 "" H 6790 3230 60  0000 C CNN
 	1    6790 3230
@@
 F 0 "MX2:3" H 7890 3340 50  0000 C CNN
 F 1 "MX2:8" H 7740 3150 50  0000 C CNN
-F 2 "idle-hands:MX_FLIP_CUTOUT" H 7740 3230 60  0001 C CNN
+F 2 "idle-hands:MX_CUTOUT_VERT" H 7740 3230 60  0001 C CNN
 F 3 "" H 7740 3230 60  0000 C CNN
 	1    7740 3230
@@
 F 0 "MX2:4" H 8840 3340 50  0000 C CNN
 F 1 "MX2:7" H 8690 3150 50  0000 C CNN
-F 2 "idle-hands:MX_FLIP_CUTOUT" H 8690 3230 60  0001 C CNN
+F 2 "idle-hands:MX_CUTOUT_VERT" H 8690 3230 60  0001 C CNN
 F 3 "" H 8690 3230 60  0000 C CNN
 	1    8690 3230
@@
 F 0 "MX3:1" H 6040 4090 50  0000 C CNN
 F 1 "MX3:10" H 5890 3900 50  0000 C CNN
-F 2 "idle-hands:MX_FLIP_CUTOUT" H 5890 3980 60  0001 C CNN
+F 2 "idle-hands:MX_CUTOUT_VERT" H 5890 3980 60  0001 C CNN
 F 3 "" H 5890 3980 60  0000 C CNN
 	1    5890 3980
@@
 F 0 "MX3:2" H 6940 4090 50  0000 C CNN
 F 1 "MX3:9" H 6790 3900 50  0000 C CNN
-F 2 "idle-hands:MX_FLIP_CUTOUT" H 6790 3980 60  0001 C CNN
+F 2 "idle-hands:MX_CUTOUT_VERT" H 6790 3980 60  0001 C CNN
 F 3 "" H 6790 3980 60  0000 C CNN
 	1    6790 3980
@@
 F 0 "MX3:3" H 7890 4090 50  0000 C CNN
 F 1 "MX3:8" H 7740 3900 50  0000 C CNN
-F 2 "idle-hands:MX_FLIP_CUTOUT" H 7740 3980 60  0001 C CNN
+F 2 "idle-hands:MX_CUTOUT_VERT" H 7740 3980 60  0001 C CNN
 F 3 "" H 7740 3980 60  0000 C CNN
 	1    7740 3980
@@
 F 0 "MX3:4" H 8840 4090 50  0000 C CNN
 F 1 "MX3:7" H 8690 3900 50  0000 C CNN
-F 2 "idle-hands:MX_FLIP_CUTOUT" H 8690 3980 60  0001 C CNN
+F 2 "idle-hands:MX_CUTOUT_VERT" H 8690 3980 60  0001 C CNN
 F 3 "" H 8690 3980 60  0000 C CNN
 	1    8690 3980
@@
 F 0 "J1" H 2930 2540 50  0000 C CNN
 F 1 "TRRS" H 3100 2090 50  0000 C CNN
-F 2 "idle-hands:PJ320D_DOUBLESIDED" H 3230 2560 50  0001 C CNN
+F 2 "Connectors:PJ320D_3.5mm_Jack" H 3230 2560 50  0001 C CNN
 F 3 "" H 3230 2560 50  0001 C CNN
 	1    2980 2460
@@
 F 0 "MX3:0" H 5140 4090 50  0000 C CNN
 F 1 "MX3:11" H 4990 3900 50  0000 C CNN
-F 2 "idle-hands:MX_FLIP_CUTOUT" H 4990 3980 60  0001 C CNN
+F 2 "idle-hands:MX_CUTOUT_VERT" H 4990 3980 60  0001 C CNN
 F 3 "" H 4990 3980 60  0000 C CNN
 	1    4990 3980
@@
 F 0 "MX1:5" H 9790 2590 50  0000 C CNN
 F 1 "MX1:6" H 9640 2400 50  0000 C CNN
-F 2 "idle-hands:MX_FLIP_CUTOUT" H 9640 2480 60  0001 C CNN
+F 2 "idle-hands:MX_CUTOUT_VERT" H 9640 2480 60  0001 C CNN
 F 3 "" H 9640 2480 60  0000 C CNN
 	1    9640 2480
@@
 F 0 "MX0:5" H 9790 1840 50  0000 C CNN
 F 1 "MX0:6" H 9640 1650 50  0000 C CNN
-F 2 "idle-hands:MX_FLIP_CUTOUT" H 9640 1730 60  0001 C CNN
+F 2 "idle-hands:MX_CUTOUT_VERT_PAD1" H 9640 1730 60  0001 C CNN
 F 3 "" H 9640 1730 60  0000 C CNN
 	1    9640 1730
@@
 F 0 "MX2:5" H 9790 3340 50  0000 C CNN
 F 1 "MX2:6" H 9640 3150 50  0000 C CNN
-F 2 "idle-hands:MX_FLIP_CUTOUT" H 9640 3230 60  0001 C CNN
+F 2 "idle-hands:MX_CUTOUT_VERT" H 9640 3230 60  0001 C CNN
 F 3 "" H 9640 3230 60  0000 C CNN
 	1    9640 3230
@@
 F 0 "MX3:5" H 9790 4090 50  0000 C CNN
 F 1 "MX3:6" H 9640 3900 50  0000 C CNN
-F 2 "idle-hands:MX_FLIP_CUTOUT" H 9640 3980 60  0001 C CNN
+F 2 "idle-hands:MX_CUTOUT_VERT" H 9640 3980 60  0001 C CNN
 F 3 "" H 9640 3980 60  0000 C CNN
 	1    9640 3980
@@
 F 0 "J2" H 2130 2500 50  0000 C CNN
 F 1 "TRRS" H 2300 2050 50  0000 C CNN
-F 2 "idle-hands:PJ320D_DOUBLESIDED" H 2430 2520 50  0001 C CNN
+F 2 "Connectors:PJ320D_3.5mm_Jack" H 2430 2520 50  0001 C CNN
 F 3 "" H 2430 2520 50  0001 C CNN
 	1    2180 2420
@@
 F 0 "MX4:1" H 6040 4820 50  0000 C CNN
 F 1 "MX4:10" H 5890 4630 50  0000 C CNN
-F 2 "idle-hands:MX_FLIP_CUTOUT" H 5890 4710 60  0001 C CNN
+F 2 "idle-hands:MX2U_CUTOUT_VERT" H 5890 4710 60  0001 C CNN
 F 3 "" H 5890 4710 60  0000 C CNN
 	1    5890 4710
@@
 F 0 "MX4:2" H 6940 4820 50  0000 C CNN
 F 1 "MX4:9" H 6790 4630 50  0000 C CNN
-F 2 "idle-hands:MX_FLIP_CUTOUT" H 6790 4710 60  0001 C CNN
+F 2 "idle-hands:MX_CUTOUT_VERT" H 6790 4710 60  0001 C CNN
 F 3 "" H 6790 4710 60  0000 C CNN
 	1    6790 4710
@@
 F 0 "MX4:3" H 7890 4820 50  0000 C CNN
 F 1 "MX4:8" H 7740 4630 50  0000 C CNN
-F 2 "idle-hands:MX_FLIP_CUTOUT" H 7740 4710 60  0001 C CNN
+F 2 "idle-hands:MX_CUTOUT_VERT" H 7740 4710 60  0001 C CNN
 F 3 "" H 7740 4710 60  0000 C CNN
 	1    7740 4710
@@
 F 0 "MX4:4" H 8840 4820 50  0000 C CNN
 F 1 "MX4:7" H 8690 4630 50  0000 C CNN
-F 2 "idle-hands:MX_FLIP_CUTOUT" H 8690 4710 60  0001 C CNN
+F 2 "idle-hands:MX2U_CUTOUT_VERT" H 8690 4710 60  0001 C CNN
 F 3 "" H 8690 4710 60  0000 C CNN
 	1    8690 4710
@@
 F 0 "MX4:0" H 5140 4820 50  0000 C CNN
 F 1 "MX4:11" H 4990 4630 50  0000 C CNN
-F 2 "idle-hands:MX_FLIP_CUTOUT" H 4990 4710 60  0001 C CNN
+F 2 "idle-hands:MX" H 4990 4710 60  0001 C CNN
 F 3 "" H 4990 4710 60  0000 C CNN
 	1    4990 4710
@@
 F 0 "MX4:5" H 9790 4820 50  0000 C CNN
 F 1 "MX4:6" H 9640 4630 50  0000 C CNN
-F 2 "idle-hands:MX_FLIP_CUTOUT" H 9640 4710 60  0001 C CNN
+F 2 "idle-hands:MX" H 9640 4710 60  0001 C CNN
 F 3 "" H 9640 4710 60  0000 C CNN
 	1    9640 4710
@@
 $EndComp
 $Comp
-L Conn_01x01 EXTRADATA
+L Conn_01x01 EXTRADATA1
 U 1 1 5A8082B9
 P 2630 1940
-F 0 "EXTRADATA" H 2630 2040 50  0000 C CNN
+F 0 "EXTRADATA1" H 2630 2040 50  0000 C CNN
 F 1 "ExtraData" H 2630 1840 50  0000 C CNN
 F 2 "canadian_footprints:SIngle_Pad" H 2630 1940 50  0001 C CNN

Commit message: Add routes for indicator LEDs
Parts:
- added L1:0, L1:1, L1:2, L1:3, L2:0, L2:1, L2:2, L2:3: LED, idle-hands:MX_LED, symbol LED
- added R1, R2: R, Resistors_THT:R_Axial_DIN0207_L6.3mm_D2.5mm_P10.16mm_Horizontal, symbol R
Connections:
- net VCC: now also R1.1, R2.1
- net LED2: now reaches U1.17 (PD1)
- net LED2: now also L2:0.1 (K), L2:1.1 (K), L2:2.1 (K), L2:3.1 (K)
- net LED1: now reaches U1.20 (PC6)
- net LED1: now also L1:0.1 (K), L1:1.1 (K), L1:2.1 (K), L1:3.1 (K)
- new net: L1:0.2 (A), L1:1.2 (A), L1:2.2 (A), L1:3.2 (A), R1.2
- new net: L2:0.2 (A), L2:1.2 (A), L2:2.2 (A), L2:3.2 (A), R2.2
- no-connect marks 8 -> 6
Changed lines of the file:
@@
 	-1   0    0    1
 $EndComp
-Wire Wire Line
-	3510 2660 3180 2660
-Wire Wire Line
-	3510 3150 3510 2660
-Connection ~ 5290 3630
-Connection ~ 5290 2880
-Connection ~ 5290 2130
-Connection ~ 8390 1730
-Connection ~ 7440 1730
-Connection ~ 6490 1730
-Connection ~ 5590 1730
-Connection ~ 4690 1730
-Connection ~ 5590 2480
-Connection ~ 6490 2480
-Connection ~ 7440 2480
-Connection ~ 8390 2480
-Connection ~ 8390 3230
-Wire Wire Line
-	8390 1380 8390 4710
-Connection ~ 7440 3230
-Wire Wire Line
-	7440 1380 7440 3980
-Connection ~ 6490 3230
-Connection ~ 5590 3230
-Wire Wire Line
-	5590 1380 5590 4710
-Connection ~ 4690 2480
-Connection ~ 6190 4380
-Connection ~ 8040 4380
-Connection ~ 7090 4380
-Connection ~ 6190 3630
-Connection ~ 8040 3630
-Connection ~ 7090 3630
-Wire Wire Line
-	4500 3630 9940 3630
-Connection ~ 6190 2130
-Connection ~ 8040 2130
-Connection ~ 7090 2130
-Wire Wire Line
-	4490 2130 9940 2130
-Connection ~ 6190 2880
-Connection ~ 8040 2880
-Connection ~ 7090 2880
-Wire Wire Line
-	4500 4380 9940 4380
 $Comp
 L SWITCH_PUSH MX3:0
@@
 	1    0    0    -1
 $EndComp
-Connection ~ 4690 3230
-Wire Wire Line
-	4690 1380 4690 4710
-Connection ~ 5290 4380
-Wire Wire Line
-	4490 2880 9940 2880
-Wire Wire Line
-	6490 1380 6490 4710
 $Comp
 L SWITCH_PUSH MX1:5
@@
 Text Label 9340 1380 2    60   ~ 0
 Col5
-Connection ~ 9340 1730
-Connection ~ 9340 2480
-Connection ~ 9340 3230
-Wire Wire Line
-	9340 1380 9340 4710
-Connection ~ 8990 4380
-Connection ~ 8990 3630
-Connection ~ 8990 2880
-Connection ~ 8990 2130
 $Comp
 L ProMicro U1
@@
 Text Label 2630 4470 0    60   ~ 0
 Col5
-Wire Wire Line
-	2630 3570 3000 3570
 $Comp
 L GND #PWR04
@@
 NoConn ~ 2630 3770
 NoConn ~ 2630 3870
-NoConn ~ 1630 4070
-NoConn ~ 1630 3770
 NoConn ~ 1630 3470
 NoConn ~ 1630 3670
 NoConn ~ 1630 3570
 NoConn ~ 2630 3370
-Wire Wire Line
-	3510 3150 1190 3150
-Wire Wire Line
-	1190 3870 1630 3870
-Connection ~ 2990 3570
-Wire Wire Line
-	1190 3150 1190 3870
 $Comp
 L Audio-Jack-4 J2
@@
 	1    0    0    -1
 $EndComp
-Wire Wire Line
-	2380 2620 2380 3150
-Connection ~ 2380 3150
 $Comp
 L VCC #PWR07
@@
 Text Label 4500 5110 2    60   ~ 0
 Row4
-Connection ~ 6190 5110
-Connection ~ 8040 5110
-Connection ~ 7090 5110
-Wire Wire Line
-	4500 5110 9940 5110
 $Comp
 L SWITCH_PUSH MX4:0
@@
 	1    0    0    -1
 $EndComp
-Connection ~ 5290 5110
 $Comp
 L SWITCH_PUSH MX4:5
@@
 	0    1    1    0
 $EndComp
-Connection ~ 8990 5110
-Connection ~ 9340 3980
-Connection ~ 8390 3980
-Wire Wire Line
-	7440 4710 7440 3970
-Connection ~ 7440 3970
-Connection ~ 6490 3980
-Connection ~ 5590 3980
-Connection ~ 4690 3980
 Text Label 1630 4470 2    60   ~ 0
 Row4
@@
 	0    -1   -1   0
 $EndComp
+$Comp
+L R R1
+U 1 1 5A900E6D
+P 1770 5470
+F 0 "R1" V 1850 5470 50  0000 C CNN
+F 1 "R" V 1770 5470 50  0000 C CNN
+F 2 "Resistors_THT:R_Axial_DIN0207_L6.3mm_D2.5mm_P10.16mm_Horizontal" V 1700 5470 50  0001 C CNN
+F 3 "" H 1770 5470 50  0001 C CNN
+	1    1770 5470
+	0    1    1    0
+$EndComp
+$Comp
+L VCC #PWR08
+U 1 1 5A9012EA
+P 1920 5470
+F 0 "#PWR08" H 1920 5320 50  0001 C CNN
+F 1 "VCC" H 1920 5620 50  0000 C CNN
+F 2 "" H 1920 5470 50  0001 C CNN
+F 3 "" H 1920 5470 50  0001 C CNN
+	1    1920 5470
+	0    1    1    0
+$EndComp
+Text Label 1240 5470 2    60   ~ 0
+LED1
+Text Label 1630 4070 2    60   ~ 0
+LED1
+Text Label 1630 3770 2    60   ~ 0
+LED2
+$Comp
+L LED L1:0
+U 1 1 5A900AED
+P 1470 4970
+F 0 "L1:0" H 1470 5070 50  0000 C CNN
+F 1 "LED" H 1470 4870 50  0000 C CNN
+F 2 "idle-hands:MX_LED" H 1470 4970 50  0001 C CNN
+F 3 "" H 1470 4970 50  0001 C CNN
+	1    1470 4970
+	1    0    0    -1
+$EndComp
+$Comp
+L LED L1:1
+U 1 1 5A903DAB
+P 1470 5300
+F 0 "L1:1" H 1470 5400 50  0000 C CNN
+F 1 "LED" H 1470 5200 50  0000 C CNN
+F 2 "idle-hands:MX_LED" H 1470 5300 50  0001 C CNN
+F 3 "" H 1470 5300 50  0001 C CNN
+	1    1470 5300
+	1    0    0    -1
+$EndComp
+Wire Wire Line
+	3510 2660 3180 2660
+Wire Wire Line
+	3510 3150 3510 2660
+Connection ~ 5290 3630
+Connection ~ 5290 2880
+Connection ~ 5290 2130
+Connection ~ 8390 1730
+Connection ~ 7440 1730
+Connection ~ 6490 1730
+Connection ~ 5590 1730
+Connection ~ 4690 1730
+Connection ~ 5590 2480
+Connection ~ 6490 2480
+Connection ~ 7440 2480
+Connection ~ 8390 2480
+Connection ~ 8390 3230
+Wire Wire Line
+	8390 1380 8390 4710
+Connection ~ 7440 3230
+Wire Wire Line
+	7440 1380 7440 3980
+Connection ~ 6490 3230
+Connection ~ 5590 3230
+Wire Wire Line
+	5590 1380 5590 4710
+Connection ~ 4690 2480
+Connection ~ 6190 4380
+Connection ~ 8040 4380
+Connection ~ 7090 4380
+Connection ~ 6190 3630
+Connection ~ 8040 3630
+Connection ~ 7090 3630
+Wire Wire Line
+	4500 3630 9940 3630
+Connection ~ 6190 2130
+Connection ~ 8040 2130
+Connection ~ 7090 2130
+Wire Wire Line
+	4490 2130 9940 2130
+Connection ~ 6190 2880
+Connection ~ 8040 2880
+Connection ~ 7090 2880
+Wire Wire Line
+	4500 4380 9940 4380
+Connection ~ 4690 3230
+Wire Wire Line
+	4690 1380 4690 4710
+Connection ~ 5290 4380
+Wire Wire Line
+	4490 2880 9940 2880
+Wire Wire Line
+	6490 1380 6490 4710
+Connection ~ 9340 1730
+Connection ~ 9340 2480
+Connection ~ 9340 3230
+Wire Wire Line
+	9340 1380 9340 4710
+Connection ~ 8990 4380
+Connection ~ 8990 3630
+Connection ~ 8990 2880
+Connection ~ 8990 2130
+Wire Wire Line
+	2630 3570 3000 3570
+Wire Wire Line
+	3510 3150 1190 3150
+Wire Wire Line
+	1190 3870 1630 3870
+Connection ~ 2990 3570
+Wire Wire Line
+	1190 3150 1190 3870
+Wire Wire Line
+	2380 2620 2380 3150
+Connection ~ 2380 3150
+Connection ~ 6190 5110
+Connection ~ 8040 5110
+Connection ~ 7090 5110
+Wire Wire Line
+	4500 5110 9940 5110
+Connection ~ 5290 5110
+Connection ~ 8990 5110
+Connection ~ 9340 3980
+Connection ~ 8390 3980
+Wire Wire Line
+	7440 4710 7440 3970
+Connection ~ 7440 3970
+Connection ~ 6490 3980
+Connection ~ 5590 3980
+Connection ~ 4690 3980
 Wire Wire Line
 	2380 2420 2630 2420
@@
 	3180 2250 2630 2250
 Connection ~ 2630 2250
+Wire Wire Line
+	1620 4970 1620 5960
+Connection ~ 1620 5470
+Wire Wire Line
+	1320 4970 1320 5960
+Wire Wire Line
+	1240 5470 1320 5470
+Wire Wire Line
+	1320 5470 1320 5460
+Connection ~ 1320 5460
+$Comp
+L R R2
+U 1 1 5A9055FD
+P 3270 5490
+F 0 "R2" V 3350 5490 50  0000 C CNN
+F 1 "R" V 3270 5490 50  0000 C CNN
+F 2 "Resistors_THT:R_Axial_DIN0207_L6.3mm_D2.5mm_P10.16mm_Horizontal" V 3200 5490 50  0001 C CNN
+F 3 "" H 3270 5490 50  0001 C CNN
+	1    3270 5490
+	0    1    1    0
+$EndComp
+$Comp
+L VCC #PWR09
+U 1 1 5A905603
+P 3420 5490
+F 0 "#PWR09" H 3420 5340 50  0001 C CNN
+F 1 "VCC" H 3420 5640 50  0000 C CNN
+F 2 "" H 3420 5490 50  0001 C CNN
+F 3 "" H 3420 5490 50  0001 C CNN
+	1    3420 5490
+	0    1    1    0
+$EndComp
+Text Label 2740 5490 2    60   ~ 0
+LED2
+$Comp
+L LED L2:0
+U 1 1 5A90560A
+P 2970 4960
+F 0 "L2:0" H 2970 5060 50  0000 C CNN
+F 1 "LED" H 2970 4860 50  0000 C CNN
+F 2 "idle-hands:MX_LED" H 2970 4960 50  0001 C CNN
+F 3 "" H 2970 4960 50  0001 C CNN
+	1    2970 4960
+	1    0    0    -1
+$EndComp
+$Comp
+L LED L2:1
+U 1 1 5A905610
+P 2970 5320
+F 0 "L2:1" H 2970 5420 50  0000 C CNN
+F 1 "LED" H 2970 5220 50  0000 C CNN
+F 2 "idle-hands:MX_LED" H 2970 5320 50  0001 C CNN
+F 3 "" H 2970 5320 50  0001 C CNN
+	1    2970 5320
+	1    0    0    -1
+$EndComp
+Wire Wire Line
+	3120 4960 3120 6000
+Connection ~ 3120 5490
+Wire Wire Line
+	2820 4960 2820 6000
+Wire Wire Line
+	2740 5490 2820 5490
+Wire Wire Line
+	2820 5490 2820 5480
+Connection ~ 2820 5480
+$Comp
+L LED L1:2
+U 1 1 5A9075D6
+P 1470 5640
+F 0 "L1:2" H 1470 5740 50  0000 C CNN
+F 1 "LED" H 1470 5540 50  0000 C CNN
+F 2 "idle-hands:MX_LED" H 1470 5640 50  0001 C CNN
+F 3 "" H 1470 5640 50  0001 C CNN
+	1    1470 5640
+	1    0    0    -1
+$EndComp
+$Comp
+L LED L1:3
+U 1 1 5A9076D0
+P 1470 5960
+F 0 "L1:3" H 1470 6060 50  0000 C CNN
+F 1 "LED" H 1470 5860 50  0000 C CNN
+F 2 "idle-hands:MX_LED" H 1470 5960 50  0001 C CNN
+F 3 "" H 1470 5960 50  0001 C CNN
+	1    1470 5960
+	1    0    0    -1
+$EndComp
+Connection ~ 1320 5300
+Connection ~ 1620 5300
+Connection ~ 1620 5640
+Connection ~ 1320 5640
+$Comp
+L LED L2:2
+U 1 1 5A908C0D
+P 2970 5660
+F 0 "L2:2" H 2970 5760 50  0000 C CNN
+F 1 "LED" H 2970 5560 50  0000 C CNN
+F 2 "idle-hands:MX_LED" H 2970 5660 50  0001 C CNN
+F 3 "" H 2970 5660 50  0001 C CNN
+	1    2970 5660
+	1    0    0    -1
+$EndComp
+$Comp
+L LED L2:3
+U 1 1 5A908D0F
+P 2970 6000
+F 0 "L2:3" H 2970 6100 50  0000 C CNN
+F 1 "LED" H 2970 5900 50  0000 C CNN
+F 2 "idle-hands:MX_LED" H 2970 6000 50  0001 C CNN
+F 3 "" H 2970 6000 50  0001 C CNN
+	1    2970 6000
+	1    0    0    -1
+$EndComp
+Connection ~ 2820 5320
+Connection ~ 3120 5320
+Connection ~ 3120 5660
+Connection ~ 2820 5660
 $EndSCHEMATC
